Commit message: update robot wheel alignment

File: src/my_robot/urdf/my_robot.xacro (robot description, xacro)
@@ -88,5 +88,5 @@
    </link>
   <joint type="continuous" name="left_wheel_hinge">
-    <origin xyz="0 0.15 0" rpy="0 0 0"/>
+    <origin xyz="0 0.125 0" rpy="0 0 0"/>
     <child link="left_wheel"/>
     <parent link="chassis"/>
@@ -115,5 +115,5 @@
    </link>
   <joint type="continuous" name="right_wheel_hinge">
-    <origin xyz="0 -0.15 0" rpy="0 0 0"/>
+    <origin xyz="0 -0.125 0" rpy="0 0 0"/>
     <child link="right_wheel"/>
     <parent link="chassis"/>
